Commit message: Spawn Robot in Gazebo

File: description/robot_core.xacro (robot description, xacro)
@@ -1,5 +1,5 @@
 <?xml version="1.0"?>
-<robot xmlns:xacro="http://www.ros.org/wiki/xacro" >
-    <xacro:include filename="inertial_macros.xacro"/>
+<robot xmlns:xacro="http://www.ros.org/wiki/xacro">
+    <xacro:include filename="inertial_macros.xacro" />
     <!-- Colours -->
     <material name="white">
@@ -20,75 +20,125 @@
     <!-- Chasis Link -->
     <joint name="chassis_joint" type="fixed">
-        <parent link="base_link"/>
-        <child link="chassis_link"/>
+        <parent link="base_link" />
+        <child link="chassis_link" />
         <origin xyz="0 0 0" />
     </joint>
     <link name="chassis_link">
         <visual>
-            <origin xyz="0.15 0 0.075"/>
+            <origin xyz="0.15 0 0.075" />
             <geometry>
-                <box size="0.3 0.3 0.15"/>
+                <box size="0.3 0.3 0.15" />
             </geometry>
-            <material name="white"/>
+            <material name="white" />
         </visual>
         <collision>
-            <origin xyz="0.15 0 0.075"/>
+            <origin xyz="0.15 0 0.075" />
             <geometry>
-                <box size="0.3 0.3 0.15"/>
+                <box size="0.3 0.3 0.15" />
             </geometry>
         </collision>
         <xacro:inertial_box mass="0.5" x="0.3" y="0.3" z="0.15">
-            <origin xyz="0.15 0 0.075" rpy="0 0 0"/>
+            <origin xyz="0.15 0 0.075" rpy="0 0 0" />
         </xacro:inertial_box>
     </link>
-    <!-- Left Wheel Link -->
-    <joint name="left_wheel_joint" type="continuous">
-        <origin xyz="0 0.175 0" rpy="-${pi/2} 0 0"/>
-        <parent link="base_link"/>
-        <child link="left_wheel_link"/>
-        <axis xyz="0 0 1"/>
+    <!-- Front Left Wheel Link -->
+    <joint name="front_left_wheel_joint" type="continuous">
+        <origin xyz="0.3 0.175 0" rpy="-${pi/2} 0 0" />
+        <parent link="base_link" />
+        <child link="front_left_wheel_link" />
+        <axis xyz="0 0 1" />
     </joint>
-    <link name="left_wheel_link">
+    <link name="front_left_wheel_link">
         <visual>
-            <origin xyz="0 0 0" rpy="0 0 0"/>
+            <origin xyz="0 0 0" rpy="0 0 0" />
             <geometry>
-                <cylinder radius="0.05" length="0.04"/>
+                <cylinder radius="0.05" length="0.04" />
             </geometry>
-            <material name="blue"/>
+            <material name="blue" />
         </visual>
         <collision>
-            <origin xyz="0 0 0" rpy="0 0 0"/>
+            <origin xyz="0 0 0" rpy="0 0 0" />
             <geometry>
-                <cylinder radius="0.05" length="0.04"/>
+                <cylinder radius="0.05" length="0.04" />
             </geometry>
         </collision>
         <xacro:inertial_cylinder mass="0.1" length="0.04" radius="0.05">
-            <origin xyz="0 0 0" rpy="0 0 0"/>
+            <origin xyz="0 0 0" rpy="0 0 0" />
         </xacro:inertial_cylinder>
     </link>
-        <!-- Right Wheel Link -->
-        <joint name="right_wheel_joint" type="continuous">
-            <origin xyz="0 -0.175 0" rpy="${pi/2} 0 0"/>
-            <parent link="base_link"/>
-            <child link="right_wheel_link"/>
-            <axis xyz="0 0 -1"/>
-        </joint>
-        <link name="right_wheel_link">
-            <visual>
-                <origin xyz="0 0 0" rpy="0 0 0"/>
-                <geometry>
-                    <cylinder radius="0.05" length="0.04"/>
-                </geometry>
-                <material name="blue"/>
-            </visual>
-            <collision>
-                <origin xyz="0 0 0" rpy="0 0 0"/>
-                <geometry>
-                    <cylinder radius="0.05" length="0.04"/>
-                </geometry>
-            </collision>
-            <xacro:inertial_cylinder mass="0.1" length="0.04" radius="0.05">
-                <origin xyz="0 0 0" rpy="0 0 0"/>
-            </xacro:inertial_cylinder>
-        </link>
+    <!-- Front Right Wheel Link -->
+    <joint name="front_right_wheel_joint" type="continuous">
+        <origin xyz="0.3 -0.175 0" rpy="${pi/2} 0 0" />
+        <parent link="base_link" />
+        <child link="front_right_wheel_link" />
+        <axis xyz="0 0 -1" />
+    </joint>
+    <link name="front_right_wheel_link">
+        <visual>
+            <origin xyz="0 0 0" rpy="0 0 0" />
+            <geometry>
+                <cylinder radius="0.05" length="0.04" />
+            </geometry>
+            <material name="blue" />
+        </visual>
+        <collision>
+            <origin xyz="0 0 0" rpy="0 0 0" />
+            <geometry>
+                <cylinder radius="0.05" length="0.04" />
+            </geometry>
+        </collision>
+        <xacro:inertial_cylinder mass="0.1" length="0.04" radius="0.05">
+            <origin xyz="0 0 0" rpy="0 0 0" />
+        </xacro:inertial_cylinder>
+    </link>
+    <!-- Rear Left Wheel Link -->
+    <joint name="rear_left_wheel_joint" type="continuous">
+        <origin xyz="0 0.175 0" rpy="-${pi/2} 0 0" />
+        <parent link="base_link" />
+        <child link="rear_left_wheel_link" />
+        <axis xyz="0 0 1" />
+    </joint>
+    <link name="rear_left_wheel_link">
+        <visual>
+            <origin xyz="0 0 0" rpy="0 0 0" />
+            <geometry>
+                <cylinder radius="0.05" length="0.04" />
+            </geometry>
+            <material name="blue" />
+        </visual>
+        <collision>
+            <origin xyz="0 0 0" rpy="0 0 0" />
+            <geometry>
+                <cylinder radius="0.05" length="0.04" />
+            </geometry>
+        </collision>
+        <xacro:inertial_cylinder mass="0.1" length="0.04" radius="0.05">
+            <origin xyz="0 0 0" rpy="0 0 0" />
+        </xacro:inertial_cylinder>
+    </link>
+    <!-- Rear Right Wheel Link -->
+    <joint name="rear_right_wheel_joint" type="continuous">
+        <origin xyz="0 -0.175 0" rpy="${pi/2} 0 0" />
+        <parent link="base_link" />
+        <child link="rear_right_wheel_link" />
+        <axis xyz="0 0 -1" />
+    </joint>
+    <link name="rear_right_wheel_link">
+        <visual>
+            <origin xyz="0 0 0" rpy="0 0 0" />
+            <geometry>
+                <cylinder radius="0.05" length="0.04" />
+            </geometry>
+            <material name="blue" />
+        </visual>
+        <collision>
+            <origin xyz="0 0 0" rpy="0 0 0" />
+            <geometry>
+                <cylinder radius="0.05" length="0.04" />
+            </geometry>
+        </collision>
+        <xacro:inertial_cylinder mass="0.1" length="0.04" radius="0.05">
+            <origin xyz="0 0 0" rpy="0 0 0" />
+        </xacro:inertial_cylinder>
+    </link>
 </robot>

Commit message: Working Gazebo

File: description/robot_core.xacro (robot description, xacro)
@@ -54,5 +54,5 @@
     <link name="chassis_link">
         <visual>
-            <origin xyz="0 0 ${-chassis_height/2}"/>
+            <origin xyz="0 0 ${chassis_height/2}"/>
             <geometry>
                 <box size="${chassis_length} ${chassis_width} ${chassis_height}"/>
