Commit message: URDF Properties Update

File: description/robot.urdf.xacro (robot description, xacro)
@@ -1,4 +1,14 @@
 <?xml version="1.0"?>
 <robot xmlns:xacro="http://www.ros.org/wiki/xacro"  name="robot">
+<!--     <xacro:arg name="use_ros2_control" default="true"/>
+    <xacro:arg name="sim_mode" default="false"/> -->
     <xacro:include filename="robot_core.xacro" />
+<!--     <xacro:if value="$(arg use_ros2_control)">
+        <xacro:include filename="ros2_control.xacro" />
+    </xacro:if>
+    <xacro:unless value="$(arg use_ros2_control)">
+        <xacro:include filename="gz_control.xacro" />
+    </xacro:unless>
+    <xacro:include filename="lidar.xacro" />
+    <xacro:include filename="camera.xacro" /> -->
 </robot>

File: description/robot_core.xacro (robot description, xacro)
@@ -2,14 +2,34 @@
 <robot xmlns:xacro="http://www.ros.org/wiki/xacro">
     <xacro:include filename="inertial_macros.xacro" />
+    <!-- Properties -->
+    <!-- Chassis -->
+    <xacro:property name="chassis_length" value="0.300"/>
+    <xacro:property name="chassis_width" value="0.200"/>
+    <xacro:property name="chassis_height" value="0.130"/>
+    <xacro:property name="chassis_mass" value="1.0"/>
+    <xacro:property name="chassis_offset_x" value="${chassis_length/2}"/>
+    <xacro:property name="chassis_offset_y" value="0"/>
+    <xacro:property name="chassis_offset_z" value="0"/>
+    <!-- Wheels -->
+    <xacro:property name="wheel_radius" value="0.065"/>
+    <xacro:property name="wheel_thickness" value="0.030"/>
+    <xacro:property name="wheel_mass" value="0.050"/>
+    <xacro:property name="wheel_offset_x" value="0.100"/>
+    <xacro:property name="wheel_offset_y" value="${(chassis_width+wheel_thickness)/2}"/>
+    <xacro:property name="wheel_offset_z" value="0.010"/>
     <!-- Colours -->
+    <!-- White -->
     <material name="white">
         <color rgba="1 1 1 1" />
     </material>
+    <!-- Orange -->
     <material name="orange">
         <color rgba="1 0.3 0.1 1" />
     </material>
+    <!-- Blue -->
     <material name="blue">
         <color rgba="0.2 0.2 1 1" />
     </material>
+    <!-- Black -->
     <material name="black">
         <color rgba="0 0 0 1" />
@@ -18,32 +38,43 @@
     <link name="base_link">
     </link>
+    <!-- Base Footprint -->
+    <joint name="base_footprint_joint" type="fixed">
+        <parent link="base_link"/>
+        <child link="base_footprint"/>
+        <origin xyz="0 0 0" rpy="0 0 0"/>
+    </joint>
+    <link name="base_footprint">
+    </link>
     <!-- Chasis Link -->
     <joint name="chassis_joint" type="fixed">
-        <parent link="base_link" />
-        <child link="chassis_link" />
-        <origin xyz="0 0 0" />
+        <parent link="base_link"/>
+        <child link="chassis_link"/>
+        <origin xyz="${chassis_offset_x} ${chassis_offset_y} ${chassis_offset_z}"/>
     </joint>
     <link name="chassis_link">
         <visual>
-            <origin xyz="0.15 0 0.075" />
+            <origin xyz="0 0 ${-chassis_height/2}"/>
             <geometry>
-                <box size="0.3 0.3 0.15" />
+                <box size="${chassis_length} ${chassis_width} ${chassis_height}"/>
             </geometry>
-            <material name="white" />
+            <material name="white"/>
         </visual>
         <collision>
-            <origin xyz="0.15 0 0.075" />
+            <origin xyz="0 0 ${-chassis_height/2}"/>
             <geometry>
-                <box size="0.3 0.3 0.15" />
+                <box size="${chassis_length} ${chassis_width} ${chassis_height}"/>
             </geometry>
         </collision>
-        <xacro:inertial_box mass="0.5" x="0.3" y="0.3" z="0.15">
-            <origin xyz="0.15 0 0.075" rpy="0 0 0" />
+        <xacro:inertial_box mass="${chassis_mass}" x="${chassis_length}" y="${chassis_width}" z="${chassis_height}">
+            <origin xyz="0 0 ${-chassis_height/2}" rpy="0 0 0"/>
         </xacro:inertial_box>
     </link>
+    <gazebo reference="chassis">
+        <material>Gazebo/White</material>
+    </gazebo>
     <!-- Front Left Wheel Link -->
     <joint name="front_left_wheel_joint" type="continuous">
-        <origin xyz="0.3 0.175 0" rpy="-${pi/2} 0 0" />
-        <parent link="base_link" />
+        <origin xyz="${wheel_offset_x} ${wheel_offset_y} ${-wheel_offset_z}" rpy="-${pi/2} 0 0" />
+        <parent link="chassis_link" />
         <child link="front_left_wheel_link" />
         <axis xyz="0 0 1" />
@@ -53,5 +84,5 @@
             <origin xyz="0 0 0" rpy="0 0 0" />
             <geometry>
-                <cylinder radius="0.05" length="0.04" />
+                <cylinder radius="${wheel_radius}" length="${wheel_thickness}" />
             </geometry>
             <material name="blue" />
@@ -60,15 +91,20 @@
             <origin xyz="0 0 0" rpy="0 0 0" />
             <geometry>
-                <cylinder radius="0.05" length="0.04" />
+                <cylinder radius="${wheel_radius}" length="${wheel_thickness}" />
             </geometry>
         </collision>
-        <xacro:inertial_cylinder mass="0.1" length="0.04" radius="0.05">
+        <xacro:inertial_cylinder mass="${wheel_mass}" length="${wheel_thickness}" radius="${wheel_radius}">
             <origin xyz="0 0 0" rpy="0 0 0" />
         </xacro:inertial_cylinder>
     </link>
+    <gazebo reference="front_left_wheel">
+        <material>
+            Gazebo/Blue
+        </material>
+    </gazebo>
     <!-- Front Right Wheel Link -->
     <joint name="front_right_wheel_joint" type="continuous">
-        <origin xyz="0.3 -0.175 0" rpy="${pi/2} 0 0" />
-        <parent link="base_link" />
+        <origin xyz="${wheel_offset_x} ${-wheel_offset_y} ${-wheel_offset_z}" rpy="${pi/2} 0 0" />
+        <parent link="chassis_link" />
         <child link="front_right_wheel_link" />
         <axis xyz="0 0 -1" />
@@ -78,5 +114,5 @@
             <origin xyz="0 0 0" rpy="0 0 0" />
             <geometry>
-                <cylinder radius="0.05" length="0.04" />
+                <cylinder radius="${wheel_radius}" length="${wheel_thickness}" />
             </geometry>
             <material name="blue" />
@@ -85,15 +121,20 @@
             <origin xyz="0 0 0" rpy="0 0 0" />
             <geometry>
-                <cylinder radius="0.05" length="0.04" />
+                <cylinder radius="${wheel_radius}" length="${wheel_thickness}" />
             </geometry>
         </collision>
-        <xacro:inertial_cylinder mass="0.1" length="0.04" radius="0.05">
+        <xacro:inertial_cylinder mass="${wheel_mass}" length="${wheel_thickness}" radius="${wheel_radius}">
             <origin xyz="0 0 0" rpy="0 0 0" />
         </xacro:inertial_cylinder>
     </link>
+    <gazebo reference="front_right_wheel">
+        <material>
+            Gazebo/Blue
+        </material>
+    </gazebo>
     <!-- Rear Left Wheel Link -->
     <joint name="rear_left_wheel_joint" type="continuous">
-        <origin xyz="0 0.175 0" rpy="-${pi/2} 0 0" />
-        <parent link="base_link" />
+        <origin xyz="${-wheel_offset_x} ${wheel_offset_y} ${-wheel_offset_z}" rpy="-${pi/2} 0 0" />
+        <parent link="chassis_link" />
         <child link="rear_left_wheel_link" />
         <axis xyz="0 0 1" />
@@ -103,5 +144,5 @@
             <origin xyz="0 0 0" rpy="0 0 0" />
             <geometry>
-                <cylinder radius="0.05" length="0.04" />
+                <cylinder radius="${wheel_radius}" length="${wheel_thickness}" />
             </geometry>
             <material name="blue" />
@@ -110,15 +151,20 @@
             <origin xyz="0 0 0" rpy="0 0 0" />
             <geometry>
-                <cylinder radius="0.05" length="0.04" />
+                <cylinder radius="${wheel_radius}" length="${wheel_thickness}" />
             </geometry>
         </collision>
-        <xacro:inertial_cylinder mass="0.1" length="0.04" radius="0.05">
+        <xacro:inertial_cylinder mass="${wheel_mass}" length="${wheel_thickness}" radius="${wheel_radius}">
             <origin xyz="0 0 0" rpy="0 0 0" />
         </xacro:inertial_cylinder>
     </link>
+    <gazebo reference="rear_left_wheel">
+        <material>
+            Gazebo/Blue
+        </material>
+    </gazebo>
     <!-- Rear Right Wheel Link -->
     <joint name="rear_right_wheel_joint" type="continuous">
-        <origin xyz="0 -0.175 0" rpy="${pi/2} 0 0" />
-        <parent link="base_link" />
+        <origin xyz="${-wheel_offset_x} ${-wheel_offset_y} ${-wheel_offset_z}" rpy="${pi/2} 0 0" />
+        <parent link="chassis_link" />
         <child link="rear_right_wheel_link" />
         <axis xyz="0 0 -1" />
@@ -128,5 +174,5 @@
             <origin xyz="0 0 0" rpy="0 0 0" />
             <geometry>
-                <cylinder radius="0.05" length="0.04" />
+                <cylinder radius="${wheel_radius}" length="${wheel_thickness}" />
             </geometry>
             <material name="blue" />
@@ -135,10 +181,15 @@
             <origin xyz="0 0 0" rpy="0 0 0" />
             <geometry>
-                <cylinder radius="0.05" length="0.04" />
+                <cylinder radius="${wheel_radius}" length="${wheel_thickness}" />
             </geometry>
         </collision>
-        <xacro:inertial_cylinder mass="0.1" length="0.04" radius="0.05">
+        <xacro:inertial_cylinder mass="${wheel_mass}" length="${wheel_thickness}" radius="${wheel_radius}">
             <origin xyz="0 0 0" rpy="0 0 0" />
         </xacro:inertial_cylinder>
     </link>
+    <gazebo reference="rear_right_wheel">
+        <material>
+            Gazebo/Blue
+        </material>
+    </gazebo>
 </robot>

Commit message: Include of FWS Controller

File: description/robot.urdf.xacro (robot description, xacro)
@@ -4,4 +4,5 @@
     <xacro:arg name="sim_mode" default="false"/> -->
     <xacro:include filename="robot_core.xacro" />
+    <xacro:include filename="ros2_control.xacro" />
     <!-- <xacro:include filename="gz_control.xacro" /> -->
 <!--     <xacro:if value="$(arg use_ros2_control)">

File: description/ros2_control.xacro (robot description, xacro)
@@ -1,36 +1,7 @@
 <?xml version="1.0"?>
 <robot xmlns:xacro="http://www.ros.org/wiki/xacro">
-    <!--     <xacro:unless value="$(arg sim_mode)">
-        <ros2_control name="RealRobot" type="system">
-            <hardware>
-                <plugin>diffdrive_arduino/DiffDriveArduino</plugin>
-                <param name="left_wheel_name">left_wheel_joint</param>
-                <param name="right_wheel_name">right_wheel_joint</param>
-                <param name="loop_rate">30</param>
-                <param name="device">/dev/ttyUSB0</param>
-                <param name="baud_rate">57600</param>
-                <param name="timeout">1000</param>
-                <param name="enc_counts_per_rev">3436</param>
-            </hardware>
-            <joint name="left_wheel_joint">
-                <command_interface name="velocity">
-                    <param name="min">-10</param>
-                    <param name="max">10</param>
-                </command_interface>
-                <state_interface name="velocity"/>
-                <state_interface name="position"/>
-            </joint>
-            <joint name="right_wheel_joint">
-                <command_interface name="velocity">
-                    <param name="min">-10</param>
-                    <param name="max">10</param>
-                </command_interface>
-                <state_interface name="velocity"/>
-                <state_interface name="position"/>
-            </joint>
-        </ros2_control>
-    </xacro:unless> -->
-    <xacro:if value="$(arg sim_mode)">
-        <ros2_control name="IgnitionSystem" type="system">
+    <!-- ROS2 Control Macro -->
+    <xacro:macro name="fws_ros2_control" params="name prefix">
+        <ros2_control name="${name}" type="system">
             <!-- Hardware -->
             <hardware>
@@ -38,34 +9,39 @@
             </hardware>
             <!-- Joints -->
-            <joint name="front_left_wheel_joint">
+            <joint name="${prefix}_steering_joint">
+                <command_interface name="position">
+                    <param name="min">{-2*pi}</param>
+                    <param name="max">{2*pi}</param>
+                </command_interface>
                 <command_interface name="velocity">
-                    <param name="min">-1</param>
-                    <param name="max">1</param>
+                    <param name="min">-3.15</param>
+                    <param name="max">3.15</param>
                 </command_interface>
+                <state_interface name="position">
+                    <param name="initial_value">0.0</param>
+                </state_interface>
                 <state_interface name="velocity" />
             </joint>
-            <joint name="front_right_wheel_joint">
+            <joint name="${prefix}_wheel_joint">
+                <command_interface name="position">
+                    <param name="min">{-2*pi}</param>
+                    <param name="max">{2*pi}</param>
+                </command_interface>
                 <command_interface name="velocity">
-                    <param name="min">-1</param>
-                    <param name="max">1</param>
+                    <param name="min">-3.15</param>
+                    <param name="max">3.15</param>
                 </command_interface>
-                <state_interface name="velocity" />
-            </joint>
-            <joint name="rear_left_wheel_joint">
-                <command_interface name="velocity">
-                    <param name="min">-1</param>
-                    <param name="max">1</param>
-                </command_interface>
-                <state_interface name="velocity" />
-            </joint>
-            <joint name="rear_right_wheel_joint">
-                <command_interface name="velocity">
-                    <param name="min">-1</param>
-                    <param name="max">1</param>
-                </command_interface>
+                <state_interface name="position">
+                    <param name="initial_value">0.0</param>
+                </state_interface>
                 <state_interface name="velocity" />
             </joint>
         </ros2_control>
-    </xacro:if>
+    </xacro:macro>
+    <!-- ROS2 Control -->
+    <xacro:fws_ros2_control name="IgnitionSystem" prefix="front_left" />
+    <xacro:fws_ros2_control name="IgnitionSystem" prefix="front_right" />
+    <xacro:fws_ros2_control name="IgnitionSystem" prefix="rear_left" />
+    <xacro:fws_ros2_control name="IgnitionSystem" prefix="rear_right" />
     <!-- Ignition Gazebo -->
     <gazebo>

Commit message: Package Built with Bicycle Steering Controller

File: description/robot.urdf.xacro (robot description, xacro)
@@ -12,5 +12,5 @@
         <xacro:include filename="gz_control.xacro" />
     </xacro:unless> -->
-    <xacro:include filename="lidar.xacro" />
-    <xacro:include filename="camera.xacro" />
+    <!-- <xacro:include filename="lidar.xacro" />
+    <xacro:include filename="camera.xacro" /> -->
 </robot>

File: description/robot_core.xacro (robot description, xacro)
@@ -59,5 +59,5 @@
     <xacro:wheel_joint prefix="rear_right" left="-1" />
     <!-- ============================= Transmission ============================= -->
-    <transmission name="steer_front_left_wheel">
+    <!-- <transmission name="steer_front_left_wheel">
         <type>transmission_interface/SimpleTransmission</type>
         <joint name="front_left_steering_joint">
@@ -78,4 +78,4 @@
             <mechanicalReduction>1</mechanicalReduction>
         </actuator>
-    </transmission>
+    </transmission> -->
 </robot>

File: description/ros2_control.xacro (robot description, xacro)
@@ -10,30 +10,18 @@
             <!-- Joints -->
             <joint name="${prefix}_steering_joint">
-                <command_interface name="position">
+                <command_interface name="steering_position">
                     <param name="min">{-2*pi}</param>
                     <param name="max">{2*pi}</param>
                 </command_interface>
-                <command_interface name="velocity">
+                <state_interface name="steering_position">
+                    <param name="initial_value">0.0</param>
+                </state_interface>
+            </joint>
+            <joint name="${prefix}_wheel_joint">
+                <command_interface name="wheel_velocity">
                     <param name="min">-3.15</param>
                     <param name="max">3.15</param>
                 </command_interface>
-                <state_interface name="position">
-                    <param name="initial_value">0.0</param>
-                </state_interface>
-                <state_interface name="velocity" />
-            </joint>
-            <joint name="${prefix}_wheel_joint">
-                <command_interface name="position">
-                    <param name="min">{-2*pi}</param>
-                    <param name="max">{2*pi}</param>
-                </command_interface>
-                <command_interface name="velocity">
-                    <param name="min">-3.15</param>
-                    <param name="max">3.15</param>
-                </command_interface>
-                <state_interface name="position">
-                    <param name="initial_value">0.0</param>
-                </state_interface>
-                <state_interface name="velocity" />
+                <state_interface name="wheel_velocity" />
             </joint>
         </ros2_control>

Commit message: Formatting and Removal of Files

File: description/robot.urdf.xacro (robot description, xacro)
@@ -1,15 +1,16 @@
 <?xml version="1.0"?>
 <robot xmlns:xacro="http://www.ros.org/wiki/xacro" name="robot">
-    <!--     <xacro:arg name="use_ros2_control" default="true"/>
-    <xacro:arg name="sim_mode" default="false"/> -->
+    <!-- Arguments -->
+    <xacro:arg name="use_ros2_control" default="true" />
+    <xacro:arg name="sim_mode" default="true" />
+    <!-- Robot Description -->
     <xacro:include filename="robot_core.xacro" />
-    <xacro:include filename="ros2_control.xacro" />
-    <!-- <xacro:include filename="gz_control.xacro" /> -->
-    <!--     <xacro:if value="$(arg use_ros2_control)">
+    <xacro:if value="$(arg use_ros2_control)">
         <xacro:include filename="ros2_control.xacro" />
     </xacro:if>
     <xacro:unless value="$(arg use_ros2_control)">
         <xacro:include filename="gz_control.xacro" />
-    </xacro:unless> -->
+    </xacro:unless>
+    <!-- Sensors -->
     <!-- <xacro:include filename="lidar.xacro" />
     <xacro:include filename="camera.xacro" /> -->

File: description/robot_core.xacro (robot description, xacro)
@@ -58,24 +58,3 @@
     <xacro:wheel_joint prefix="rear_left" left="1" />
     <xacro:wheel_joint prefix="rear_right" left="-1" />
-    <!-- ============================= Transmission ============================= -->
-    <!-- <transmission name="steer_front_left_wheel">
-        <type>transmission_interface/SimpleTransmission</type>
-        <joint name="front_left_steering_joint">
-            <hardwareInterface>EffortJointInterface</hardwareInterface>
-        </joint>
-        <actuator name="motor_front_left_steering">
-            <hardwareInterface>EffortJointInterface</hardwareInterface>
-            <mechanicalReduction>1</mechanicalReduction>
-        </actuator>
-    </transmission>
-    <transmission name="drive_front_left_wheel">
-        <type>transmission_interface/SimpleTransmission</type>
-        <joint name="front_left_wheel_joint">
-            <hardwareInterface>EffortJointInterface</hardwareInterface>
-        </joint>
-        <actuator name="motor_front_left_wheel">
-            <hardwareInterface>EffortJointInterface</hardwareInterface>
-            <mechanicalReduction>1</mechanicalReduction>
-        </actuator>
-    </transmission> -->
 </robot>

File: description/ros2_control.xacro (robot description, xacro)
@@ -10,18 +10,18 @@
             <!-- Joints -->
             <joint name="${prefix}_steering_joint">
-                <command_interface name="steering_position">
-                    <param name="min">{-2*pi}</param>
-                    <param name="max">{2*pi}</param>
+                <command_interface name="position">
+                    <param name="min">{-pi/4}</param>
+                    <param name="max">{pi/4}</param>
                 </command_interface>
-                <state_interface name="steering_position">
-                    <param name="initial_value">0.0</param>
-                </state_interface>
+                <state_interface name="position" />
+                <state_interface name="velocity" />
             </joint>
             <joint name="${prefix}_wheel_joint">
-                <command_interface name="wheel_velocity">
-                    <param name="min">-3.15</param>
-                    <param name="max">3.15</param>
+                <command_interface name="velocity">
+                    <param name="min">-10</param>
+                    <param name="max">10</param>
                 </command_interface>
-                <state_interface name="wheel_velocity" />
+                <state_interface name="position" />
+                <state_interface name="velocity" />
             </joint>
         </ros2_control>
@@ -37,5 +37,5 @@
         <plugin filename="ign_ros2_control-system"
             name="ign_ros2_control::IgnitionROS2ControlPlugin">
-            <parameters>$(find park_bot)/config/fws_controller.yaml</parameters>
+            <parameters>$(find park_bot)/config/my_controller.yaml</parameters>
         </plugin>
     </gazebo>
