Commit message: Working Update RSP

File: description/ros2_control.xacro (robot description, xacro)
@@ -1,5 +1,5 @@
 <?xml version="1.0"?>
 <robot xmlns:xacro="http://www.ros.org/wiki/xacro">
-    <xacro:unless value="$(arg sim_mode)">
+    <!--     <xacro:unless value="$(arg sim_mode)">
         <ros2_control name="RealRobot" type="system">
             <hardware>
@@ -30,32 +30,48 @@
             </joint>
         </ros2_control>
-    </xacro:unless>
+    </xacro:unless> -->
     <xacro:if value="$(arg sim_mode)">
-        <ros2_control name="GazeboSystem" type="system">
+        <ros2_control name="IgnitionSystem" type="system">
+            <!-- Hardware -->
             <hardware>
-                <plugin>gazebo_ros2_control/GazeboSystem</plugin>
+                <plugin>ign_ros2_control/IgnitionSystem</plugin>
             </hardware>
-            <joint name="left_wheel_joint">
+            <!-- Joints -->
+            <joint name="front_left_wheel_joint">
                 <command_interface name="velocity">
-                    <param name="min">-10</param>
-                    <param name="max">10</param>
+                    <param name="min">-1</param>
+                    <param name="max">1</param>
                 </command_interface>
-                <state_interface name="velocity"/>
-                <state_interface name="position"/>
+                <state_interface name="velocity" />
             </joint>
-            <joint name="right_wheel_joint">
+            <joint name="front_right_wheel_joint">
                 <command_interface name="velocity">
-                    <param name="min">-10</param>
-                    <param name="max">10</param>
+                    <param name="min">-1</param>
+                    <param name="max">1</param>
                 </command_interface>
-                <state_interface name="velocity"/>
-                <state_interface name="position"/>
+                <state_interface name="velocity" />
+            </joint>
+            <joint name="rear_left_wheel_joint">
+                <command_interface name="velocity">
+                    <param name="min">-1</param>
+                    <param name="max">1</param>
+                </command_interface>
+                <state_interface name="velocity" />
+            </joint>
+            <joint name="rear_right_wheel_joint">
+                <command_interface name="velocity">
+                    <param name="min">-1</param>
+                    <param name="max">1</param>
+                </command_interface>
+                <state_interface name="velocity" />
             </joint>
         </ros2_control>
     </xacro:if>
+    <!-- Ignition Gazebo -->
     <gazebo>
-        <plugin name="gazebo_ros2_control" filename="libgazebo_ros2_control.so">
-            <parameters>$(find articubot_one)/config/my_controllers.yaml</parameters>
-            <parameters>$(find articubot_one)/config/gaz_ros2_ctl_use_sim.yaml</parameters>
+        <!-- Joint State Publisher -->
+        <plugin filename="ign_ros2_control-system"
+            name="ign_ros2_control::IgnitionROS2ControlPlugin">
+            <parameters>$(find park_bot)/config/fws_controller.yaml</parameters>
         </plugin>
     </gazebo>

Commit message: Working JointGroup(Position/Velocity)Controllers

File: description/ros2_control.xacro (robot description, xacro)
@@ -2,34 +2,28 @@
 <robot xmlns:xacro="http://www.ros.org/wiki/xacro">
     <!-- ROS2 Control Macro -->
-    <xacro:macro name="fws_ros2_control" params="name prefix">
-        <ros2_control name="${name}" type="system">
-            <!-- Hardware -->
-            <hardware>
-                <plugin>ign_ros2_control/IgnitionSystem</plugin>
-            </hardware>
-            <!-- Joints -->
-            <joint name="${prefix}_steering_joint">
-                <command_interface name="position">
-                    <param name="min">{-pi/4}</param>
-                    <param name="max">{pi/4}</param>
-                </command_interface>
-                <state_interface name="position" />
-                <state_interface name="velocity" />
-            </joint>
-            <joint name="${prefix}_wheel_joint">
-                <command_interface name="velocity">
-                    <param name="min">-10</param>
-                    <param name="max">10</param>
-                </command_interface>
-                <state_interface name="position" />
-                <state_interface name="velocity" />
-            </joint>
-        </ros2_control>
+    <xacro:macro name="fws_ros2_control" params="prefix">
+        <!-- Hardware -->
+        <hardware>
+            <plugin>ign_ros2_control/IgnitionSystem</plugin>
+        </hardware>
+        <!-- Joints -->
+        <joint name="${prefix}_steering_joint">
+            <command_interface name="position" />
+            <state_interface name="position" />
+            <state_interface name="velocity" />
+        </joint>
+        <joint name="${prefix}_wheel_joint">
+            <command_interface name="velocity" />
+            <state_interface name="position" />
+            <state_interface name="velocity" />
+        </joint>
     </xacro:macro>
     <!-- ROS2 Control -->
-    <xacro:fws_ros2_control name="IgnitionSystem" prefix="front_left" />
-    <xacro:fws_ros2_control name="IgnitionSystem" prefix="front_right" />
-    <xacro:fws_ros2_control name="IgnitionSystem" prefix="rear_left" />
-    <xacro:fws_ros2_control name="IgnitionSystem" prefix="rear_right" />
+    <ros2_control name="IgnitionSystem" type="system">
+        <xacro:fws_ros2_control prefix="front_left" />
+        <xacro:fws_ros2_control prefix="front_right" />
+        <xacro:fws_ros2_control prefix="rear_left" />
+        <xacro:fws_ros2_control prefix="rear_right" />
+    </ros2_control>
     <!-- Ignition Gazebo -->
     <gazebo>
