Commit message: LIDAR Launch File

File: description/camera.xacro (robot description, xacro)
@@ -1,20 +1,22 @@
 <?xml version="1.0"?>
 <robot xmlns:xacro="http://www.ros.org/wiki/xacro" >
+    <!-- Properties -->
+    <!-- Camera -->
+    <xacro:property name="camera_offset_x" value="${chassis_length/2}"/>
+    <xacro:property name="camera_offset_y" value="0"/>
+    <xacro:property name="camera_offset_z" value="${chassis_height/2}"/>
+    <xacro:property name="camera_radius" value="0.010"/>
+    <xacro:property name="camera_thickness" value="0.03"/>
+    <!-- Camera Link -->
     <joint name="camera_joint" type="fixed">
         <parent link="chassis_link"/>
         <child link="camera_link"/>
-        <origin xyz="0.276 0 0.181" rpy="0 0.18 0"/>
+        <origin xyz="0.15 0 0.065" rpy="0 0 0"/>
     </joint>
     <link name="camera_link">
         <visual>
+            <origin xyz="${camera_thickness/2} 0 0" rpy="0 ${pi/2} 0"/>
             <geometry>
-                <box size="0.010 0.03 0.03"/>
-            </geometry>
-            <material name="black"/>
-        </visual>
-        <visual>
-            <origin xyz="0 0 -0.05"/>
-            <geometry>
-                <cylinder radius="0.002" length="0.1"/>
+                <cylinder radius="${camera_radius}" length="${camera_thickness}"/>
             </geometry>
             <material name="black"/>
@@ -33,4 +35,5 @@
             <visualize>true</visualize>
             <update_rate>10</update_rate>
+            <topic>camerae</topic>
             <camera>
                 <horizontal_fov>1.089</horizontal_fov>
@@ -45,7 +48,5 @@
                 </clip>
             </camera>
-            <plugin name="camera_controller" filename="libgazebo_ros_camera.so">
-                <frame_name>camera_link_optical</frame_name>
-            </plugin>
+            <plugin filename="ignition-gazebo-sensors-system" name="gz::sim::systems::Sensors"></plugin>
         </sensor>
     </gazebo>

File: description/robot.urdf.xacro (robot description, xacro)
@@ -11,5 +11,5 @@
         <xacro:include filename="gz_control.xacro" />
     </xacro:unless>
-    <xacro:include filename="lidar.xacro" />
-    <xacro:include filename="camera.xacro" /> -->
+    <xacro:include filename="lidar.xacro" /> -->
+    <xacro:include filename="camera.xacro" />
 </robot>

Commit message: Correct Camera LiDAR URDF

File: description/camera.xacro (robot description, xacro)
@@ -3,18 +3,15 @@
     <!-- Properties -->
     <!-- Camera -->
-    <xacro:property name="camera_offset_x" value="${chassis_length/2}"/>
-    <xacro:property name="camera_offset_y" value="0"/>
-    <xacro:property name="camera_offset_z" value="${chassis_height/2}"/>
-    <xacro:property name="camera_radius" value="0.010"/>
-    <xacro:property name="camera_thickness" value="0.03"/>
-    <!-- Camera Link -->
+    <xacro:property name="camera_offset_x" value="${(chassis_length+camera_thickness)/2}"/>
+    <xacro:property name="camera_radius" value="0.015"/>
+    <xacro:property name="camera_thickness" value="0.01"/>
     <joint name="camera_joint" type="fixed">
         <parent link="chassis_link"/>
         <child link="camera_link"/>
-        <origin xyz="0.15 0 0.065" rpy="0 0 0"/>
+        <origin xyz="${camera_offset_x} 0 0" rpy="0 ${pi/2} 0"/>
     </joint>
     <link name="camera_link">
         <visual>
-            <origin xyz="${camera_thickness/2} 0 0" rpy="0 ${pi/2} 0"/>
+            <origin xyz="0 0 0" rpy="0 0 0"/>
             <geometry>
                 <cylinder radius="${camera_radius}" length="${camera_thickness}"/>
@@ -35,5 +32,5 @@
             <visualize>true</visualize>
             <update_rate>10</update_rate>
-            <topic>camerae</topic>
+            <topic>camera</topic>
             <camera>
                 <horizontal_fov>1.089</horizontal_fov>

File: description/lidar.xacro (robot description, xacro)
@@ -1,20 +1,18 @@
 <?xml version="1.0"?>
 <robot xmlns:xacro="http://www.ros.org/wiki/xacro" >
+    <xacro:include filename="properties.xacro"/>
+    <xacro:property name="laser_offset_z" value="${(chassis_height+laser_thickness)/2}"/>
+    <xacro:property name="laser_radius" value="0.02"/>
+    <xacro:property name="laser_thickness" value="0.01"/>
+    <xacro:property name="laser_mass" value="0.1"/>
     <joint name="laser_joint" type="fixed">
         <parent link="chassis_link"/>
         <child link="laser_frame"/>
-        <origin xyz="0 0 0.212" rpy="0 0 0"/>
+        <origin xyz="0 0 ${laser_offset_z}" rpy="0 0 0"/>
     </joint>
     <link name="laser_frame">
         <visual>
             <geometry>
-                <cylinder radius="0.05" length="0.04"/>
-            </geometry>
-            <material name="black"/>
-        </visual>
-        <visual>
-            <origin xyz="0 0 -0.05"/>
-            <geometry>
-                <cylinder radius="0.01" length="0.1"/>
+                <cylinder radius="${laser_radius}" length="${laser_thickness}"/>
             </geometry>
             <material name="black"/>
@@ -22,8 +20,8 @@
         <collision>
             <geometry>
-                <cylinder radius="0.05" length="0.04"/>
+                <cylinder radius="${laser_radius}" length="${laser_thickness}"/>
             </geometry>
         </collision>
-        <xacro:inertial_cylinder mass="0.1" length="0.04" radius="0.05">
+        <xacro:inertial_cylinder mass="${laser_mass}" length="${laser_thickness}" radius="${laser_radius}">
             <origin xyz="0 0 0" rpy="0 0 0"/>
         </xacro:inertial_cylinder>

File: description/robot.urdf.xacro (robot description, xacro)
@@ -11,5 +11,5 @@
         <xacro:include filename="gz_control.xacro" />
     </xacro:unless> -->
-    <!-- <xacro:include filename="lidar.xacro" />
-    <xacro:include filename="camera.xacro" />  -->
+    <xacro:include filename="lidar.xacro" />
+    <xacro:include filename="camera.xacro" />
 </robot>

Commit message: Working LiDAR

File: description/camera.xacro (robot description, xacro)
@@ -45,5 +45,5 @@
                 </clip>
             </camera>
-            <plugin filename="ignition-gazebo-sensors-system" name="gz::sim::systems::Sensors"></plugin>
+            <plugin filename="gz-sim-sensors-system" name="gz::sim::systems::Sensors"></plugin>
         </sensor>
     </gazebo>

File: description/lidar.xacro (robot description, xacro)
@@ -27,43 +27,18 @@
             <origin xyz="0 0 0" rpy="0 0 0" />
         </xacro:inertial_cylinder>
-        <sensor name='lidar' type='lidar'>
-            <topic>lidar</topic>
+    </link>
+    <!-- Ignition Gazebo -->
+    <gazebo reference="laser_frame">
+        <material>Gazebo/Black</material>
+        <sensor name="laser" type="gpu_lidar">
+            <pose>0 0 0 0 0 0</pose>
+            <topic>scan</topic>
+            <visualize>true</visualize>
             <update_rate>10</update_rate>
             <lidar>
                 <scan>
                     <horizontal>
-                        <samples>640</samples>
+                        <samples>360</samples>
                         <resolution>1</resolution>
-                        <min_angle>-1.396263</min_angle>
-                        <max_angle>1.396263</max_angle>
-                    </horizontal>
-                    <vertical>
-                        <samples>16</samples>
-                        <resolution>1</resolution>
-                        <min_angle>-0.261799</min_angle>
-                        <max_angle>0.261799</max_angle>
-                    </vertical>
-                </scan>
-                <range>
-                    <min>0.08</min>
-                    <max>10.0</max>
-                    <resolution>0.01</resolution>
-                </range>
-            </lidar>
-            <alwaysOn>1</alwaysOn>
-            <visualize>true</visualize>
-        </sensor>
-    </link>
-    <!-- Ignition Gazebo -->
-    <gazebo reference="laser_frame">
-        <material>Gazebo/Black</material>
-        <sensor name="laser" type="ray">
-            <pose> 0 0 0 0 0 0 </pose>
-            <visualize>true</visualize>
-            <update_rate>10</update_rate>
-            <ray>
-                <scan>
-                    <horizontal>
-                        <samples>360</samples>
                         <min_angle>-3.14</min_angle>
                         <max_angle>3.14</max_angle>
@@ -73,12 +48,13 @@
                     <min>0.3</min>
                     <max>12</max>
+                    <resolution>0.01</resolution>
                 </range>
-            </ray>
+            </lidar>
             <plugin filename="ignition-gazebo-sensors-system" name="gz::sim::systems::Sensors">
-                <ros>
+                <!-- <ros>
                     <argument>~/out:=scan</argument>
                 </ros>
-                <output_type>sensor_msgs/msg/LaserScan</output_type>
-                <frame_name>laser_frame</frame_name>
+                <output_type>sensor_msgs/LaserScan</output_type>
+                <frame_name>laser_frame</frame_name> -->
             </plugin>
         </sensor>

File: description/robot_core.xacro (robot description, xacro)
@@ -58,3 +58,19 @@
     <xacro:wheel_joint prefix="rear_left" left="1" />
     <xacro:wheel_joint prefix="rear_right" left="-1" />
+    <!-- <gazebo>
+        <plugin
+            filename="gz-sim-odometry-publisher-system"
+            name="gz::sim::systems::OdometryPublisher">
+            <odom_frame>odom</odom_frame>
+            <robot_base_frame>base_link</robot_base_frame>
+        </plugin>
+        <plugin
+            filename="gz-sim-pose-publisher-system"
+            name="gz::sim::systems::PosePublisher">
+            <publish_link_pose>true</publish_link_pose>
+            <use_pose_vector_msg>true</use_pose_vector_msg>
+            <static_publisher>true</static_publisher>
+            <static_update_frequency>1</static_update_frequency>
+        </plugin>
+    </gazebo> -->
 </robot>
