Commit message: World Updates

File: description/robot_macros.xacro (robot description, xacro)
@@ -6,14 +6,14 @@
         <link name="${prefix}_steering_link">
             <visual name="">
-                <origin xyz="0 0 0" rpy="0 0 0"/>
+                <origin xyz="0 0 0" rpy="0 0 0" />
                 <geometry>
-                    <cylinder radius="${steering_radius}" length="${steering_length}"/>
+                    <cylinder radius="${steering_radius}" length="${steering_length}" />
                 </geometry>
-                <material name="blue"/>
+                <material name="blue" />
             </visual>
             <collision>
-                <origin xyz="0 0 0" rpy="0 0 0"/>
+                <origin xyz="0 0 0" rpy="0 0 0" />
                 <geometry>
-                    <cylinder radius="${steering_radius}" length="${steering_length}"/>
+                    <cylinder radius="${steering_radius}" length="${steering_length}" />
                 </geometry>
             </collision>

File: description/ros2_control.xacro (robot description, xacro)
@@ -31,5 +31,5 @@
         <plugin filename="ign_ros2_control-system"
             name="ign_ros2_control::IgnitionROS2ControlPlugin">
-            <parameters>$(find park_bot)/config/my_controller.yaml</parameters>
+            <parameters>$(find park_bot)/config/my_controllers.yaml</parameters>
         </plugin>
     </gazebo>

Commit message: Updated Kinematics

File: description/robot_macros.xacro (robot description, xacro)
@@ -59,5 +59,5 @@
             <parent link="chassis_link" />
             <child link="${prefix}_steering_link" />
-            <axis xyz="0 ${left} 0" />
+            <axis xyz="0 ${-left} 0" />
             <limit lower="-${pi/4}" upper="${pi/4}" effort="100" velocity="1" />
         </joint>

Commit message: Good Rise Time

File: description/robot_macros.xacro (robot description, xacro)
@@ -60,5 +60,5 @@
             <child link="${prefix}_steering_link" />
             <axis xyz="0 ${-left} 0" />
-            <limit lower="-${pi/4}" upper="${pi/4}" effort="100" velocity="1" />
+            <limit lower="-${pi/4}" upper="${pi/4}" effort="100" velocity="100" />
         </joint>
     </xacro:macro>
