Commit message: Working Steering RSP

File: description/properties.xacro (robot description, xacro)
@@ -8,11 +8,16 @@
     <xacro:property name="chassis_offset_x" value="${chassis_length/2}"/>
     <xacro:property name="chassis_offset_y" value="0"/>
-    <xacro:property name="chassis_offset_z" value="0"/>
+    <xacro:property name="chassis_offset_z" value="${chassis_height/2}"/>
+    <!-- Steering -->
+    <xacro:property name="steering_radius" value="0.01"/>
+    <xacro:property name="steering_length" value="0.02"/>
+    <xacro:property name="steering_mass" value="0.01"/>
+    <xacro:property name="steering_offset_x" value="${(2/3)*chassis_length/2}"/>
+    <xacro:property name="steering_offset_y" value="${(chassis_width+steering_length)/2}"/>
+    <xacro:property name="steering_offset_z" value="${(2/3)*chassis_height/2}"/>
     <!-- Wheels -->
     <xacro:property name="wheel_radius" value="0.065"/>
     <xacro:property name="wheel_thickness" value="0.030"/>
     <xacro:property name="wheel_mass" value="0.050"/>
-    <xacro:property name="wheel_offset_x" value="0.100"/>
-    <xacro:property name="wheel_offset_y" value="${(chassis_width+wheel_thickness)/2 + 0.1}"/>
-    <xacro:property name="wheel_offset_z" value="0.010"/>
+    <xacro:property name="wheel_offset_z" value="${steering_length+wheel_thickness/2}"/>
 </robot>

File: description/robot.urdf.xacro (robot description, xacro)
@@ -11,5 +11,5 @@
         <xacro:include filename="gz_control.xacro" />
     </xacro:unless> -->
-    <xacro:include filename="lidar.xacro" />
-    <xacro:include filename="camera.xacro" />
+    <!-- <xacro:include filename="lidar.xacro" />
+    <xacro:include filename="camera.xacro" />  -->
 </robot>

File: description/robot_core.xacro (robot description, xacro)
@@ -11,5 +11,5 @@
     <link name="chassis_link">
         <visual>
-            <origin xyz="0 0 ${chassis_height/2}" />
+            <origin xyz="0 0 0" />
             <geometry>
                 <box size="${chassis_length} ${chassis_width} ${chassis_height}" />
@@ -18,5 +18,5 @@
         </visual>
         <collision>
-            <origin xyz="0 0 ${-chassis_height/2}" />
+            <origin xyz="0 0 0" />
             <geometry>
                 <box size="${chassis_length} ${chassis_width} ${chassis_height}" />
@@ -25,5 +25,5 @@
         <xacro:inertial_box mass="${chassis_mass}" x="${chassis_length}" y="${chassis_width}"
             z="${chassis_height}">
-            <origin xyz="0 0 ${-chassis_height/2}" rpy="0 0 0" />
+            <origin xyz="0 0 0" />
         </xacro:inertial_box>
     </link>
@@ -31,4 +31,9 @@
         <material>Gazebo/White</material>
     </gazebo>
+    <!-- Steering Links -->
+    <xacro:steering_link prefix="front_left" />
+    <xacro:steering_link prefix="front_right" />
+    <xacro:steering_link prefix="rear_left" />
+    <xacro:steering_link prefix="rear_right" />
     <!-- Wheel Links -->
     <xacro:wheel_link prefix="front_left" />
@@ -36,6 +41,4 @@
     <xacro:wheel_link prefix="rear_left" />
     <xacro:wheel_link prefix="rear_right" />
-    <!-- Steering Links -->
-    <link name="front_left_steering_link"/>
     <!-- ================================ Joints ================================ -->
     <!-- Chassis Joint -->
@@ -46,23 +49,33 @@
     </joint>
     <!-- Steering Joints -->
-    <xacro:steering_joint prefix="front_left" />
-    <xacro:steering_joint prefix="front_right" />
-    <xacro:steering_joint prefix="rear_left" />
-    <xacro:steering_joint prefix="rear_right" />
+    <xacro:steering_joint prefix="front_left" front="1" left="1" />
+    <xacro:steering_joint prefix="front_right" front="1" left="-1" />
+    <xacro:steering_joint prefix="rear_left" front="-1" left="1" />
+    <xacro:steering_joint prefix="rear_right" front="-1" left="-1" />
     <!-- Wheel Joints -->
-    <xacro:wheel_joint prefix="front_left" front="1" left="1" />
-    <xacro:wheel_joint prefix="front_right" front="1" left="-1" />
-    <xacro:wheel_joint prefix="rear_left" front="-1" left="1" />
-    <xacro:wheel_joint prefix="rear_right" front="-1" left="-1" />
+    <xacro:wheel_joint prefix="front_left" left="1" />
+    <xacro:wheel_joint prefix="front_right" left="-1" />
+    <xacro:wheel_joint prefix="rear_left" left="1" />
+    <xacro:wheel_joint prefix="rear_right" left="-1" />
     <!-- ============================= Transmission ============================= -->
-    <transmission name="trans_front_left_wheel_rotate">
+    <transmission name="steer_front_left_wheel">
         <type>transmission_interface/SimpleTransmission</type>
-        <joint name="front_left_rotate">
-          <hardwareInterface>EffortJointInterface</hardwareInterface>
+        <joint name="front_left_steering_joint">
+            <hardwareInterface>EffortJointInterface</hardwareInterface>
+        </joint>
+        <actuator name="motor_front_left_steering">
+            <hardwareInterface>EffortJointInterface</hardwareInterface>
+            <mechanicalReduction>1</mechanicalReduction>
+        </actuator>
+    </transmission>
+    <transmission name="drive_front_left_wheel">
+        <type>transmission_interface/SimpleTransmission</type>
+        <joint name="front_left_wheel_joint">
+            <hardwareInterface>EffortJointInterface</hardwareInterface>
         </joint>
         <actuator name="motor_front_left_wheel">
-          <hardwareInterface>EffortJointInterface</hardwareInterface>
-          <mechanicalReduction>1</mechanicalReduction>
+            <hardwareInterface>EffortJointInterface</hardwareInterface>
+            <mechanicalReduction>1</mechanicalReduction>
         </actuator>
-      </transmission>
+    </transmission>
 </robot>

File: description/robot_macros.xacro (robot description, xacro)
@@ -2,4 +2,29 @@
 <robot xmlns:xacro="http://www.ros.org/wiki/xacro">
     <xacro:include filename="properties.xacro" />
+    <!-- Steering Link -->
+    <xacro:macro name="steering_link" params="prefix">
+        <link name="${prefix}_steering_link">
+            <visual name="">
+                <origin xyz="0 0 0" rpy="0 0 0"/>
+                <geometry>
+                    <cylinder radius="${steering_radius}" length="${steering_length}"/>
+                </geometry>
+                <material name="blue"/>
+            </visual>
+            <collision>
+                <origin xyz="0 0 0" rpy="0 0 0"/>
+                <geometry>
+                    <cylinder radius="${steering_radius}" length="${steering_length}"/>
+                </geometry>
+            </collision>
+            <xacro:inertial_cylinder mass="${steering_mass}" length="${steering_length}"
+                radius="${steering_radius}">
+                <origin xyz="0 0 0" rpy="0 0 0" />
+            </xacro:inertial_cylinder>
+        </link>
+        <gazebo reference="${prefix}_steering">
+            <material>Gazebo/Blue</material>
+        </gazebo>
+    </xacro:macro>
     <!-- Wheel Link -->
     <xacro:macro name="wheel_link" params="prefix">
@@ -28,19 +53,20 @@
     </xacro:macro>
     <!-- Steering Joints -->
-    <xacro:macro name="steering_joint" params="prefix">
+    <xacro:macro name="steering_joint" params="prefix front left">
         <joint name="${prefix}_steering_joint" type="revolute">
-            <origin xyz="${wheel_offset_x} ${wheel_offset_y} -${wheel_offset_z}" rpy="0 0 0" />
+            <origin xyz="${front*steering_offset_x} ${left*steering_offset_y} -${steering_offset_z}"
+                rpy="${-1*left*pi/2} 0 0" />
             <parent link="chassis_link" />
-            <child link="${prefix}_wheel_link" />
-            <axis xyz="0 0 1" />
-            <limit lower="0" upper="${pi/4}" effort="1" velocity="1" />
+            <child link="${prefix}_steering_link" />
+            <axis xyz="0 ${left} 0" />
+            <limit lower="-${pi/4}" upper="${pi/4}" effort="100" velocity="1" />
         </joint>
     </xacro:macro>
     <!-- Wheel Joints -->
-    <xacro:macro name="wheel_joint" params="prefix front left">
+    <xacro:macro name="wheel_joint" params="prefix left">
         <joint name="${prefix}_wheel_joint" type="continuous">
-            <origin xyz="${front*wheel_offset_x} ${left*wheel_offset_y} -${wheel_offset_z}"
-                rpy="${-1*left*pi/2} 0 0" />
-            <parent link="chassis_link" />
+            <origin xyz="0 0 ${wheel_offset_z}"
+                rpy="0 0 0" />
+            <parent link="${prefix}_steering_link" />
             <child link="${prefix}_wheel_link" />
             <axis xyz="0 0 ${left}" />

Commit message: Testing for Results

File: description/properties.xacro (robot description, xacro)
@@ -2,22 +2,22 @@
 <robot xmlns:xacro="http://www.ros.org/wiki/xacro" >
     <!-- Chassis -->
-    <xacro:property name="chassis_length" value="0.300"/>
-    <xacro:property name="chassis_width" value="0.200"/>
-    <xacro:property name="chassis_height" value="0.130"/>
-    <xacro:property name="chassis_mass" value="1.0"/>
+    <xacro:property name="chassis_length" value="0.300"/>                   <!-- 0.800 -->
+    <xacro:property name="chassis_width" value="0.200"/>                    <!-- 0.400 -->
+    <xacro:property name="chassis_height" value="0.130"/>                   <!-- 0.130 -->
+    <xacro:property name="chassis_mass" value="2.0"/>                       <!-- 0.1 -->
     <xacro:property name="chassis_offset_x" value="${chassis_length/2}"/>
     <xacro:property name="chassis_offset_y" value="0"/>
     <xacro:property name="chassis_offset_z" value="${chassis_height/2}"/>
     <!-- Steering -->
-    <xacro:property name="steering_radius" value="0.01"/>
-    <xacro:property name="steering_length" value="0.02"/>
-    <xacro:property name="steering_mass" value="0.01"/>
+    <xacro:property name="steering_radius" value="0.01"/>                   <!-- 0.01 -->
+    <xacro:property name="steering_length" value="0.02"/>                   <!-- 0.01 -->
+    <xacro:property name="steering_mass" value="0.02"/>
     <xacro:property name="steering_offset_x" value="${(2/3)*chassis_length/2}"/>
     <xacro:property name="steering_offset_y" value="${(chassis_width+steering_length)/2}"/>
-    <xacro:property name="steering_offset_z" value="${(2/3)*chassis_height/2}"/>
+    <xacro:property name="steering_offset_z" value="${(2/3)*chassis_height/2}"/> <!-- 0 -->
     <!-- Wheels -->
-    <xacro:property name="wheel_radius" value="0.065"/>
-    <xacro:property name="wheel_thickness" value="0.030"/>
-    <xacro:property name="wheel_mass" value="0.050"/>
+    <xacro:property name="wheel_radius" value="0.065"/>                     <!-- 0.07 -->
+    <xacro:property name="wheel_thickness" value="0.030"/>                  <!-- 0.005 -->
+    <xacro:property name="wheel_mass" value="0.3"/>                         <!-- 1 -->
     <xacro:property name="wheel_offset_z" value="${steering_length+wheel_thickness/2}"/>
 </robot>

File: description/robot.urdf.xacro (robot description, xacro)
@@ -9,7 +9,4 @@
         <xacro:include filename="ros2_control.xacro" />
     </xacro:if>
-    <xacro:unless value="$(arg use_ros2_control)">
-        <xacro:include filename="gz_control.xacro" />
-    </xacro:unless>
     <!-- Sensors -->
     <xacro:include filename="lidar.xacro" />

File: description/robot_core.xacro (robot description, xacro)
@@ -58,4 +58,11 @@
     <xacro:wheel_joint prefix="rear_left" left="1" />
     <xacro:wheel_joint prefix="rear_right" left="-1" />
+    <!-- ================================ Gazebo ================================ -->
+    <gazebo>
+        <plugin filename="ignition-gazebo-odometry-publisher-system" name="ignition::gazebo::systems::OdometryPublisher">
+            <odom_frame>odom</odom_frame>
+            <robot_base_frame>robot/base_link</robot_base_frame>
+        </plugin>
+    </gazebo>
     <!-- <gazebo>
         <plugin

File: description/robot_macros.xacro (robot description, xacro)
@@ -25,4 +25,6 @@
         <gazebo reference="${prefix}_steering">
             <material>Gazebo/Blue</material>
+            <mu1 value="0.5" />
+            <mu2 value="0.5" />
         </gazebo>
     </xacro:macro>
@@ -50,4 +52,6 @@
         <gazebo reference="${prefix}_wheel">
             <material>Gazebo/Blue</material>
+            <mu1 value="1.0" />
+            <mu2 value="1.0" />
         </gazebo>
     </xacro:macro>
@@ -60,5 +64,5 @@
             <child link="${prefix}_steering_link" />
             <axis xyz="0 ${-left} 0" />
-            <limit lower="-${pi/4}" upper="${pi/4}" effort="100" velocity="100" />
+            <limit lower="-${pi/4}" upper="${pi/4}" effort="1" velocity="100" />
         </joint>
     </xacro:macro>
@@ -74,2 +78,23 @@
     </xacro:macro>
 </robot>
+                <!-- <surface>
+                    <friction>
+                        <ode>
+                            <mu>50.000000</mu>
+                            <mu2>50.000000</mu2>
+                            <fdir1>0.000000 0.000000 0.000000</fdir1>
+                            <slip1>0.000000</slip1>
+                            <slip2>0.000000</slip2>
+                        </ode>
+                    </friction>
+                    <contact>
+                        <ode>
+                            <soft_cfm>0.000000</soft_cfm>
+                            <soft_erp>0.200000</soft_erp>
+                            <kp>1000000000.000000</kp>
+                            <kd>1.000000</kd>
+                            <max_vel>100.000000</max_vel>
+                            <min_depth>0.001000</min_depth>
+                        </ode>
+                    </contact>
+                </surface> -->

File: description/ros2_control.xacro (robot description, xacro)
@@ -32,4 +32,5 @@
             name="ign_ros2_control::IgnitionROS2ControlPlugin">
             <parameters>$(find park_bot)/config/my_controllers.yaml</parameters>
+            <!-- <parameters>$(find park_bot)/config/vehicle_model.yaml</parameters> -->
         </plugin>
     </gazebo>

Commit message: Saved Velocity Controller

File: description/properties.xacro (robot description, xacro)
@@ -5,5 +5,5 @@
     <xacro:property name="chassis_width" value="0.200"/>                    <!-- 0.400 -->
     <xacro:property name="chassis_height" value="0.130"/>                   <!-- 0.130 -->
-    <xacro:property name="chassis_mass" value="2.0"/>                       <!-- 0.1 -->
+    <xacro:property name="chassis_mass" value="1"/>                       <!-- 0.1 -->
     <xacro:property name="chassis_offset_x" value="${chassis_length/2}"/>
     <xacro:property name="chassis_offset_y" value="0"/>

File: description/robot_macros.xacro (robot description, xacro)
@@ -42,5 +42,5 @@
                 <origin xyz="0 0 0" rpy="0 0 0" />
                 <geometry>
-                    <cylinder radius="${wheel_radius}" length="${wheel_thickness}" />
+                    <sphere radius="${wheel_radius}" />
                 </geometry>
             </collision>
@@ -50,8 +50,8 @@
             </xacro:inertial_cylinder>
         </link>
-        <gazebo reference="${prefix}_wheel">
+        <gazebo reference="${prefix}_wheel_link">
             <material>Gazebo/Blue</material>
-            <mu1 value="1.0" />
-            <mu2 value="1.0" />
+            <mu1 value="0.001"/>
+            <mu2 value="0.001" />
         </gazebo>
     </xacro:macro>
@@ -78,5 +78,5 @@
     </xacro:macro>
 </robot>
-                <!-- <surface>
+<!-- <surface>
                     <friction>
                         <ode>

Commit message: New Park World

File: description/properties.xacro (robot description, xacro)
@@ -5,5 +5,5 @@
     <xacro:property name="chassis_width" value="0.200"/>                    <!-- 0.400 -->
     <xacro:property name="chassis_height" value="0.130"/>                   <!-- 0.130 -->
-    <xacro:property name="chassis_mass" value="1"/>                       <!-- 0.1 -->
+    <xacro:property name="chassis_mass" value="1"/>                       <!-- 0.1 1 -->
     <xacro:property name="chassis_offset_x" value="${chassis_length/2}"/>
     <xacro:property name="chassis_offset_y" value="0"/>
@@ -19,5 +19,5 @@
     <xacro:property name="wheel_radius" value="0.065"/>                     <!-- 0.07 -->
     <xacro:property name="wheel_thickness" value="0.030"/>                  <!-- 0.005 -->
-    <xacro:property name="wheel_mass" value="0.3"/>                         <!-- 1 -->
+    <xacro:property name="wheel_mass" value="0.3"/>                         <!-- 1 0.3 -->
     <xacro:property name="wheel_offset_z" value="${steering_length+wheel_thickness/2}"/>
 </robot>

File: description/robot_macros.xacro (robot description, xacro)
@@ -25,6 +25,4 @@
         <gazebo reference="${prefix}_steering">
             <material>Gazebo/Blue</material>
-            <mu1 value="0.5" />
-            <mu2 value="0.5" />
         </gazebo>
     </xacro:macro>
@@ -52,6 +50,7 @@
         <gazebo reference="${prefix}_wheel_link">
             <material>Gazebo/Blue</material>
-            <mu1 value="0.001"/>
-            <mu2 value="0.001" />
+            <mu1>1.0</mu1>
+            <mu2>0.01</mu2>
+            <fdir1>0 0 1</fdir1>
         </gazebo>
     </xacro:macro>
@@ -78,23 +77,2 @@
     </xacro:macro>
 </robot>
-<!-- <surface>
-                    <friction>
-                        <ode>
-                            <mu>50.000000</mu>
-                            <mu2>50.000000</mu2>
-                            <fdir1>0.000000 0.000000 0.000000</fdir1>
-                            <slip1>0.000000</slip1>
-                            <slip2>0.000000</slip2>
-                        </ode>
-                    </friction>
-                    <contact>
-                        <ode>
-                            <soft_cfm>0.000000</soft_cfm>
-                            <soft_erp>0.200000</soft_erp>
-                            <kp>1000000000.000000</kp>
-                            <kd>1.000000</kd>
-                            <max_vel>100.000000</max_vel>
-                            <min_depth>0.001000</min_depth>
-                        </ode>
-                    </contact>
-                </surface> -->
